Commit message: fix URDF, no warning on load

File: tiago_rl/assets/tiago_strain.urdf (robot description, URDF)
Before this commit: robot tiago, 52 links, 51 joints
Links:
- removed link base_mic_back_left_link
- removed link base_mic_back_right_link
- removed link base_mic_front_left_link
- removed link base_mic_front_right_link
- link base_footprint: mass None -> 100.0
Joints:
- removed joint base_mic_back_left_joint
- removed joint base_mic_back_right_joint
- removed joint base_mic_front_left_joint
- removed joint base_mic_front_right_joint
