Commit message: deformable objects test

File: tiago_rl/assets/boxBotStrain.urdf (robot description, URDF)
Before this commit: robot boxBot, 6 links, 5 joints
Links:
- link torso: geometry visual cylinder length=0.43 radius=0.025
Joints:
- joint torso_to_arm: origin xyz=0.05 0 0.13 -> xyz=0.05 0 0.17

Commit message: lower the gripper

File: tiago_rl/assets/boxBotStrain.urdf (robot description, URDF)
Before this commit: robot boxBot, 6 links, 5 joints
Joints:
- joint torso_to_arm: origin xyz=0.05 0 0.17 -> xyz=0.05 0 0.13
