Commit message: fix notation: camelCase to snake_case

File: tiago_rl/assets/gripper_tactile.urdf (robot description, URDF)
Before this commit: robot boxBot, 6 links, 5 joints
Joints:
- joint gripper_left_finger_joint: child gripper_left_finger -> gripper_left_finger_link
- joint gripper_right_finger_joint: child gripper_right_finger -> gripper_right_finger_link

File: tiago_rl/assets/objects/object.urdf (robot description, URDF)
Before this commit: robot object, 1 links, 0 joints
Links:
- removed link objectLink
- added link object_link, mass 0.421; collision cylinder length=0.1 radius=0.02; visual cylinder length=0.1 radius=0.02

File: tiago_rl/assets/objects/table.urdf (robot description, URDF)
Before this commit: robot table, 1 links, 0 joints
Links:
- removed link tableLink
- added link table_link, mass 100.0; collision box size=0.55 0.55 0.55; visual box size=0.55 0.55 0.55

Commit message: create LoadCellVisualiser
- creates QT Plot to visualise forces

File: tiago_rl/assets/gripper_tactile.urdf (robot description, URDF)
Before this commit: robot boxBot, 6 links, 5 joints
Links:
- removed link gripper_left_finger
- removed link gripper_right_finger
- added link gripper_left_finger_link, mass 0.109980; collision box size=0.01 0.05 0.11; visual mesh filename=assets/meshes/gripper/gripper_finger_ta11_link.stl
- added link gripper_right_finger_link, mass 0.109980; collision box size=0.01 0.05 0.11; visual mesh filename=assets/meshes/gripper/gripper_finger_ta11_link.stl scale=-1 -1 1

Commit message: rename GripperEnv torso joint

File: tiago_rl/assets/gripper_tactile.urdf (robot description, URDF)
Before this commit: robot boxBot, 6 links, 5 joints
Joints:
- removed joint torso_to_arm
- added joint torso_lift_joint: type prismatic, parent torso, child arm, origin xyz=0.05 0 0.13, axis 0 0 1, limit lower=0 upper=0.05 effort=1000.0 velocity=0.5
