Commit message: REFACTOR create BulletRobotEnv and first version of GripperTactileEnv

File: tiago_rl/assets/objects/object.urdf (robot description, URDF)
Before this commit: robot cylinder, 1 links, 0 joints
Links:
- removed link cylinderLink
- added link objectLink, mass 0.421; collision cylinder length=0.1 radius=0.02; visual cylinder length=0.1 radius=0.02

File: tiago_rl/assets/objects/table.urdf (robot description, URDF)
Before this commit: robot box, 1 links, 0 joints
Links:
- removed link boxLink
- added link tableLink, mass 100.0; collision box size=0.55 0.55 0.55; visual box size=0.55 0.55 0.55

Commit message: change object stiffness

File: tiago_rl/assets/objects/object.urdf (robot description, URDF)
Before this commit: robot object, 1 links, 0 joints
Links:
- link object_link: mass 0.421 -> 2
